File: adioHAT.kicad_pcb (KiCad board)
At the start: 2 copper layers, 65 x 56 mm, 29 parts, among them J1 Conn_01x01, J2 Conn_02x02_Odd_Even, J3 Conn_02x20_Odd_Even, J4 Conn_02x20_Odd_Even, U1 AD8603, U2 AD5693RxRM, U3 AD5593R, U4 LM7321, U5 PCA9575D, U6 TXU0104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

Commit message: exchanged DAC IC
Parts:
- C7: value 10n -> 100n
- U2: value AD5693RxRM -> DAC7571; footprint Package_SO:MSOP-10_3x3mm_P0.5mm -> Package_TO_SOT_SMD:SOT-23-6
- moved C7 11.4 mm to (106.0, 64.8), turned to -90 degrees
- moved C3 6.00 mm to (113.8, 60.7), turned to 180 degrees
- moved U4 3.71 mm to (109.0, 64.6), turned to 180 degrees
- moved J1 2.95 mm to (103.4, 84.5)
- moved U2 1.57 mm to (113.7, 64.6)
Connections:
- C3 pad 2: +5V -> +3V3
- C7 pad 2: Net-(U2-VREF) -> +5V
- U2 pad 1: +5V -> Net-(U2-VOUT)
- U2 pad 2: +3V3 -> GND
- U2 pad 4: GND -> /SDA
- U2 pad 5: GND -> /SCL
Routing:
- net Net-(U2-VOUT): track 11.6 -> 2.41 mm
- net Net-(U2-VREF): track 7.55 -> 0.00 mm, vias 2 -> 0
- net GND: track 29.2 -> 35.4 mm, vias 39 -> 41
- net /VDUT: track 117.2 -> 121.3 mm, vias 1 -> 3
- net /SDA: track 58.1 -> 55.2 mm, vias 2 -> 0
- net /SCL: track 58.0 -> 59.9 mm, vias 0 -> 3
- net +5V: track 130.5 -> 128.5 mm
- net /PWM1: track 20.9 -> 21.3 mm, vias 0 -> 2
- net +3V3: track 145.8 -> 145.7 mm, vias 6 -> 5
- net Net-(U7-B4Y): track 21.5 -> 21.4 mm, vias 2 -> 0
- net Net-(U7-B1Y): vias 2 -> 0
- net Net-(U7-B2Y): vias 2 -> 0
- net Net-(U7-B3Y): vias 2 -> 0
Other:
- board text added: "DAC7571"
- board text removed: "AD5693"
